Commit message: add caster

File: catkin_ws/src/ros_robotics/urdf/dd_robot.urdf (robot description, URDF)
Before this commit: robot dd_robot, 3 links, 2 joints
Links:
- link base_link: geometry visual box size=0.5 0.5 0.25; visual sphere radius=0.05
Joints:
- joint joint_left_wheel: origin xyz=0 0.30 0 rpy=0 0 0 -> xyz=0 0.32 0 rpy=0 0 0
- joint joint_right_wheel: origin xyz=0 -0.30 0 rpy=0 0 0 -> xyz=0 -0.32 0 rpy=0 0 0
